File: ergogen/output/pcbs/corney_island.kicad_pcb (KiCad board)
At the start: 2 copper layers, 133.8 x 91.7 mm, 94 parts

Commit message: Checkpoint
Parts:
- added MH1: , ceoloide:mounting_hole_npth, F.Cu at (207.8, 100.5)
- added MH2: , ceoloide:mounting_hole_npth, F.Cu at (222.2, 109.0)
- added MH3: , ceoloide:mounting_hole_npth, F.Cu at (109.5, 71.5)
- added MH4: , ceoloide:mounting_hole_npth, F.Cu at (109.5, 90.5)
- added MH5: , ceoloide:mounting_hole_npth, F.Cu at (185.5, 68.0)
- added MH6: , ceoloide:mounting_hole_npth, F.Cu at (152.7, 107.7)
- added MH7: , ceoloide:mounting_hole_npth, F.Cu at (199.2, 115.3)
- D1, D10, D11, D12, D13, D14, D15, D16, D17, D18, D19, D2, D20, D21, D22, D23, D24, D25, D26, D27, D28, D29, D3, D30, D31, D32, D33, D34, D35, D36, D37, D38, D39, D4, D40, D41, D42, D5, D6, D7, D8, D9: footprint ComboDiode -> ceoloide:diode_tht_sod123
- DISP1: footprint combo_display -> ceoloide:display_ssd1306_nice_view
- LED1, LED10, LED11, LED12, LED13, LED14, LED15, LED16, LED17, LED18, LED19, LED2, LED20, LED21, LED3, LED4, LED5, LED6, LED7, LED8, LED9: footprint ceoloide:YS-SK6812MINI-E (per-key, reversible) -> ceoloide:led_SK6812mini-e (per-key, reversible)
- LED22, LED23, LED24, LED25, LED26, LED27: footprint ceoloide:YS-SK6812MINI-E (underglow, reversible) -> ceoloide:led_SK6812mini-e (underglow, reversible)
- MCU1: footprint nice_nano -> ceoloide:nice_nano
- RST1: renamed from B1; value Reset (PTS636 SP43 LFS) -> reset_switch_tht_top; footprint ceoloide:top-actuated-reset-switch -> ceoloide:reset_switch_tht_top
- TRRS1: footprint ceoloide:TRRS-PJ-320A-dual (reversible, symmetric) -> ceoloide:trrs_pj320a (reversible, symmetric)
- moved D41 0.40 mm to (180.7, 114.4)
- moved D21 0.40 mm to (212.3, 114.3)
- moved D42 0.40 mm to (204.9, 127.1)
- moved D1 0.40 mm to (107.4, 98.7)
- moved D10 0.40 mm to (164.4, 91.5)
- moved D11 0.40 mm to (164.4, 72.5)
- moved D12 0.40 mm to (164.4, 53.5)
- moved D13 0.40 mm to (183.4, 93.9)
- moved D14 0.40 mm to (183.4, 74.9)
- moved D15 0.40 mm to (183.4, 55.9)
- moved D16 0.40 mm to (202.4, 96.3)
- moved D17 0.40 mm to (202.4, 77.3)
- moved D18 0.40 mm to (202.4, 58.3)
- moved D19 0.40 mm to (173.9, 113.5)
- moved D2 0.40 mm to (107.4, 79.7)
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Connections:
- MCU1 pad 1: MCU1_1 -> RAW
- MCU1 pad 10: MCU1_10 -> C5
- MCU1 pad 11: MCU1_11 -> P16
- MCU1 pad 12: MCU1_12 -> P10
- MCU1 pad 13: MCU1_13 -> MCU1_12
- MCU1 pad 14: MCU1_14 -> MCU1_11
- MCU1 pad 15: MCU1_15 -> MCU1_10
- MCU1 pad 16: MCU1_16 -> MCU1_9
- MCU1 pad 17: MCU1_17 -> MCU1_8
- MCU1 pad 18: MCU1_18 -> MCU1_7
- MCU1 pad 19: MCU1_19 -> MCU1_6
- MCU1 pad 2: MCU1_2 -> GND
- MCU1 pad 20: MCU1_20 -> MCU1_5
- MCU1 pad 21: MCU1_21 -> MCU1_4
- MCU1 pad 22: MCU1_22 -> MCU1_3
- MCU1 pad 23: MCU1_23 -> MCU1_2
- MCU1 pad 24: MCU1_24 -> MCU1_1
- MCU1 pad 3: MCU1_3 -> RST
- MCU1 pad 4: MCU1_4 -> VCC
- MCU1 pad 5: MCU1_5 -> C0
- MCU1 pad 6: MCU1_6 -> C1
- MCU1 pad 7: MCU1_7 -> C2
- MCU1 pad 8: MCU1_8 -> C3
- MCU1 pad 9: MCU1_9 -> C4
Routing:
- net C0: track 121.9 -> 14.2 mm
- net C3: track 121.8 -> 14.2 mm
- net index_top: track 0.00 -> 101.6 mm
- net outer_bottom: track 0.00 -> 101.4 mm
- net DISP1_4: track 3.62 -> 0.00 mm
- net DISP1_3: track 3.62 -> 0.00 mm
- net DISP1_2: track 3.62 -> 0.00 mm
- net DISP1_1: track 3.62 -> 0.00 mm
Other:
- outline, holes or cut-outs redrawn
