File: ergogen/output/pcbs/frontplate.kicad_pcb (KiCad board)
At the start: 2 copper layers, 139.5 x 113.2 mm, 5 parts

Commit message: Checkpoint
Parts:
- moved MH5 10.00 mm to (220.8, 121.4)
Other:
- outline, holes or cut-outs redrawn
Changed lines of the file:
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@@
   )
   (module "ceoloide:mounting_hole_npth" (layer F.Cu)
-      (at 227.2307082 129.0614476 -50)
+      (at 220.8028321 121.40100319999999 -50)
       (fp_text reference "MH5" (at 0 2.55 -50) (layer F.SilkS) hide (effects (font (size 1 1) (thickness 0.15))))
       (pad "" np_thru_hole circle (at 0 0 -50) (size 2.2 2.2) (drill 2.2) (layers *.Cu *.Mask))
@@
 (gr_circle (center 185.468 61.361000000000004) (end 186.56799999999998 61.361000000000004) (layer Edge.Cuts) (width 0.15))
 (gr_circle (center 172.7442902 101.1746489) (end 173.8442902 101.1746489) (layer Edge.Cuts) (width 0.15))
-(gr_circle (center 227.2307082 129.0614476) (end 228.3307082 129.0614476) (layer Edge.Cuts) (width 0.15))
+(gr_circle (center 220.8028321 121.40100319999999) (end 221.90283209999998 121.40100319999999) (layer Edge.Cuts) (width 0.15))
 )

Commit message: Checkpoint
Other:
- board size 139.5 x 113.2 mm -> 139.4 x 113.2 mm
Changed lines of the file:
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@@
 (gr_line (start 204.08222186790144 44.61264651408419) (end 204.08299999999997 46.36499999993248) (angle 90) (layer Edge.Cuts) (width 0.15))
 (gr_line (start 204.083 46.36522199999308) (end 204.083 95.28476811661676) (angle 90) (layer Edge.Cuts) (width 0.15))
-(gr_line (start 204.333 95.71778081661677) (end 224.32222257695057 107.2585638521032) (angle 90) (layer Edge.Cuts) (width 0.15))
-(gr_line (start 224.5624582750168 107.59324544246215) (end 230.57788045934672 137.58349973883196) (angle 90) (layer Edge.Cuts) (width 0.15))
-(gr_line (start 230.40903856128045 138.06485304847308) (end 217.11551321531311 149.21944520216027) (angle 90) (layer Edge.Cuts) (width 0.15))
+(gr_line (start 204.333 95.71778081661677) (end 224.2725151534555 107.22986525776808) (angle 90) (layer Edge.Cuts) (width 0.15))
+(gr_line (start 224.52245345345548 107.6550224577677) (end 224.8868869272579 130.84827901796052) (angle 90) (layer Edge.Cuts) (width 0.15))
+(gr_line (start 225.00380302725722 131.16181731796115) (end 230.3148039002676 137.491221684766) (angle 90) (layer Edge.Cuts) (width 0.15))
+(gr_line (start 230.25317550026756 138.19563768476607) (end 217.1155132153131 149.21944520216027) (angle 90) (layer Edge.Cuts) (width 0.15))
 (gr_line (start 216.41109721531305 149.1578168021602) (end 205.28039649130588 135.89276421578668) (angle 90) (layer Edge.Cuts) (width 0.15))
 (gr_line (start 205.18757259130587 135.8069910157867) (end 189.74612938848182 124.80148031587586) (angle 90) (layer Edge.Cuts) (width 0.15))
@@
 (gr_arc (start 203.583 46.36522199999308) (end 204.083 46.36522199999308) (angle -0.025439331376729293) (layer Edge.Cuts) (width 0.15))
 (gr_arc (start 204.583 95.28476811661676) (end 204.083 95.28476811661676) (angle -59.999999891584196) (layer Edge.Cuts) (width 0.15))
-(gr_arc (start 224.07222257695054 107.69157655210316) (end 224.56245827695054 107.59324545210316) (angle -48.65815876654466) (layer Edge.Cuts) (width 0.15))
-(gr_arc (start 230.08764476128047 137.68183084847306) (end 230.40903856128048 138.06485304847305) (angle -61.34183996217147) (layer Edge.Cuts) (width 0.15))
-(gr_arc (start 216.7941194153131 148.83642300216025) (end 216.4110972153131 149.15781680216026) (angle -90.00000000000713) (layer Edge.Cuts) (width 0.15))
+(gr_arc (start 224.0225151534555 107.6628779577681) (end 224.52245345345548 107.6550224577681) (angle -59.09978888585279) (layer Edge.Cuts) (width 0.15))
+(gr_arc (start 225.38682522725793 130.84042351796052) (end 224.88688692725793 130.84827901796052) (angle -39.09979015719355) (layer Edge.Cuts) (width 0.15))
+(gr_arc (start 229.93178170026758 137.812615484766) (end 230.2531755002676 138.195637684766) (angle -90.00000000000456) (layer Edge.Cuts) (width 0.15))
+(gr_arc (start 216.79411941531308 148.83642300216025) (end 216.41109721531308 149.15781680216026) (angle -90.00000000000503) (layer Edge.Cuts) (width 0.15))
 (gr_arc (start 204.8973742913059 136.21415801578672) (end 205.2803964913059 135.8927642157867) (angle -14.521558200128908) (layer Edge.Cuts) (width 0.15))
 (gr_arc (start 189.45593108848183 125.20864731587585) (end 189.74612938848182 124.80148031587585) (angle -15.00000020686845) (layer Edge.Cuts) (width 0.15))

Commit message: Checkpoint
Other:
- board size 139.4 x 113.2 mm -> 139.3 x 113.2 mm
Changed lines of the file:
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@@
 (gr_line (start 204.08222186790144 44.61264651408419) (end 204.08299999999997 46.36499999993248) (angle 90) (layer Edge.Cuts) (width 0.15))
 (gr_line (start 204.083 46.36522199999308) (end 204.083 95.28476811661676) (angle 90) (layer Edge.Cuts) (width 0.15))
-(gr_line (start 204.333 95.71778081661677) (end 224.2725151534555 107.22986525776808) (angle 90) (layer Edge.Cuts) (width 0.15))
-(gr_line (start 224.52245345345548 107.6550224577677) (end 224.8868869272579 130.84827901796052) (angle 90) (layer Edge.Cuts) (width 0.15))
-(gr_line (start 225.00380302725722 131.16181731796115) (end 230.3148039002676 137.491221684766) (angle 90) (layer Edge.Cuts) (width 0.15))
-(gr_line (start 230.25317550026756 138.19563768476607) (end 217.1155132153131 149.21944520216027) (angle 90) (layer Edge.Cuts) (width 0.15))
+(gr_line (start 204.333 95.71778081661677) (end 224.02516425544047 107.0870571502174) (angle 90) (layer Edge.Cuts) (width 0.15))
+(gr_line (start 224.17240351287623 107.82371600590119) (end 215.00087220666293 119.82219672773476) (angle 90) (layer Edge.Cuts) (width 0.15))
+(gr_line (start 215.02579756409878 120.45958288341856) (end 230.29136629405417 137.4895566408562) (angle 90) (layer Edge.Cuts) (width 0.15))
+(gr_line (start 230.2404461940542 138.20631884085628) (end 217.11551321531311 149.21944520216024) (angle 90) (layer Edge.Cuts) (width 0.15))
 (gr_line (start 216.41109721531305 149.1578168021602) (end 205.28039649130588 135.89276421578668) (angle 90) (layer Edge.Cuts) (width 0.15))
 (gr_line (start 205.18757259130587 135.8069910157867) (end 189.74612938848182 124.80148031587586) (angle 90) (layer Edge.Cuts) (width 0.15))
@@
 (gr_arc (start 203.583 46.36522199999308) (end 204.083 46.36522199999308) (angle -0.025439331376729293) (layer Edge.Cuts) (width 0.15))
 (gr_arc (start 204.583 95.28476811661676) (end 204.083 95.28476811661676) (angle -59.999999891584196) (layer Edge.Cuts) (width 0.15))
-(gr_arc (start 224.0225151534555 107.6628779577681) (end 224.52245345345548 107.6550224577681) (angle -59.09978888585279) (layer Edge.Cuts) (width 0.15))
-(gr_arc (start 225.38682522725793 130.84042351796052) (end 224.88688692725793 130.84827901796052) (angle -39.09979015719355) (layer Edge.Cuts) (width 0.15))
-(gr_arc (start 229.93178170026758 137.812615484766) (end 230.2531755002676 138.195637684766) (angle -90.00000000000456) (layer Edge.Cuts) (width 0.15))
-(gr_arc (start 216.79411941531308 148.83642300216025) (end 216.41109721531308 149.15781680216026) (angle -90.00000000000503) (layer Edge.Cuts) (width 0.15))
+(gr_arc (start 223.77516425544044 107.52006985021737) (end 224.17240345544045 107.82371595021736) (angle -97.39397443707864) (layer Edge.Cuts) (width 0.15))
+(gr_arc (start 215.39811146409872 120.12584288341861) (end 215.00087226409872 119.82219678341862) (angle -79.2668383669675) (layer Edge.Cuts) (width 0.15))
+(gr_arc (start 229.9190523940542 137.82329664085626) (end 230.24044619405421 138.20631884085626) (angle -91.8728626585997) (layer Edge.Cuts) (width 0.15))
+(gr_arc (start 216.7941194153131 148.83642300216025) (end 216.4110972153131 149.15781680216026) (angle -90.00000000000924) (layer Edge.Cuts) (width 0.15))
 (gr_arc (start 204.8973742913059 136.21415801578672) (end 205.2803964913059 135.8927642157867) (angle -14.521558200128908) (layer Edge.Cuts) (width 0.15))
 (gr_arc (start 189.45593108848183 125.20864731587585) (end 189.74612938848182 124.80148031587585) (angle -15.00000020686845) (layer Edge.Cuts) (width 0.15))
@@
 (gr_circle (center 185.468 61.361000000000004) (end 186.56799999999998 61.361000000000004) (layer Edge.Cuts) (width 0.15))
 (gr_circle (center 172.7442902 101.1746489) (end 173.8442902 101.1746489) (layer Edge.Cuts) (width 0.15))
-(gr_circle (center 220.8028321 121.40100319999999) (end 221.90283209999998 121.40100319999999) (layer Edge.Cuts) (width 0.15))
 )
