File: ergogen/output/pcbs/frontplate.kicad_pcb (KiCad board)
At the start: 2 copper layers, 139.3 x 113.2 mm, 5 parts

Commit message: Checkpoint
Parts:
- moved MH5 10.0 mm to (214.4, 113.7)
Other:
- outline, holes or cut-outs redrawn
Changed lines of the file:
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@@
   )
   (module "ceoloide:mounting_hole_npth" (layer F.Cu)
-      (at 220.8028321 121.40100319999999 -50)
+      (at 214.374956 113.7405587 -50)
       (fp_text reference "MH5" (at 0 2.55 -50) (layer F.SilkS) hide (effects (font (size 1 1) (thickness 0.15))))
       (pad "" np_thru_hole circle (at 0 0 -50) (size 2.2 2.2) (drill 2.2) (layers *.Cu *.Mask))
@@
 (gr_circle (center 185.468 61.361000000000004) (end 186.56799999999998 61.361000000000004) (layer Edge.Cuts) (width 0.15))
 (gr_circle (center 172.7442902 101.1746489) (end 173.8442902 101.1746489) (layer Edge.Cuts) (width 0.15))
+(gr_circle (center 214.374956 113.7405587) (end 215.474956 113.7405587) (layer Edge.Cuts) (width 0.15))
 )

Commit message: Checkpoint
Parts:
- removed MH5: , ceoloide:mounting_hole_npth
Other:
- outline, holes or cut-outs redrawn
Changed lines of the file:
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@@
       (pad "" np_thru_hole circle (at 0 0 -20) (size 2.2 2.2) (drill 2.2) (layers *.Cu *.Mask))
-  )
-  (module "ceoloide:mounting_hole_npth" (layer F.Cu)
-      (at 214.374956 113.7405587 -50)
-      (fp_text reference "MH5" (at 0 2.55 -50) (layer F.SilkS) hide (effects (font (size 1 1) (thickness 0.15))))
-      (pad "" np_thru_hole circle (at 0 0 -50) (size 2.2 2.2) (drill 2.2) (layers *.Cu *.Mask))
   )
             (gr_line (start 91.08198220107948 108.73940536100417) (end 91.08001772002542 53.48837571544573) (angle 90) (layer Edge.Cuts) (width 0.15))
@@
 (gr_circle (center 185.468 61.361000000000004) (end 186.56799999999998 61.361000000000004) (layer Edge.Cuts) (width 0.15))
 (gr_circle (center 172.7442902 101.1746489) (end 173.8442902 101.1746489) (layer Edge.Cuts) (width 0.15))
-(gr_circle (center 214.374956 113.7405587) (end 215.474956 113.7405587) (layer Edge.Cuts) (width 0.15))
 )
