File: ergogen/output/pcbs/frontplate.kicad_pcb (KiCad board)
At the start: 2 copper layers, 124.2 x 110.1 mm, 5 parts

Commit message: Tweak shape
Other:
- board size 124.2 x 110.1 mm -> 124.1 x 110.1 mm
Changed lines of the file:
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@@
       (pad "" np_thru_hole circle (at 0 0 -30) (size 2.2 2.2) (drill 2.2) (layers *.Cu *.Mask))
   )
-  (gr_line (start 91.87535728883249 109.45769882370212) (end 87.06061104775414 54.447423555018986) (layer Edge.Cuts) (stroke (width 0.15) (type default)))
+  (gr_line (start 91.87827173174675 109.49099742324222) (end 87.06061104775414 54.447423555018986) (layer Edge.Cuts) (stroke (width 0.15) (type default)))
 (gr_line (start 87.51811429808367 53.90547845906503) (end 108.50503754967045 52.19601094528491) (layer Edge.Cuts) (stroke (width 0.15) (type default)))
 (gr_line (start 108.964445 51.69766144933076) (end 108.964445 39.90788282277217) (layer Edge.Cuts) (stroke (width 0.15) (type default)))
@@
 (gr_line (start 165.47394415076104 43.03997791277865) (end 183.45917122939375 42.77019950801905) (layer Edge.Cuts) (stroke (width 0.15) (type default)))
 (gr_line (start 183.96667038015485 43.26992130873259) (end 183.96744510000002 45.01459040003829) (layer Edge.Cuts) (stroke (width 0.15) (type default)))
-(gr_line (start 183.9674451 45.01481240004068) (end 183.9674451 93.93435851661681) (layer Edge.Cuts) (stroke (width 0.15) (type default)))
-(gr_line (start 184.2174451 94.36737121661682) (end 204.22421145980977 105.91828315985939) (layer Edge.Cuts) (stroke (width 0.15) (type default)))
-(gr_line (start 204.4565945725017 106.21974150639812) (end 211.26934923259248 131.20072772663832) (layer Edge.Cuts) (stroke (width 0.15) (type default)))
-(gr_line (start 211.14051951990047 131.6858354800995) (end 198.27245950682325 144.55389549317673) (layer Edge.Cuts) (stroke (width 0.15) (type default)))
+(gr_line (start 183.9674451 45.01481240004068) (end 183.9674451 88.4733585166168) (layer Edge.Cuts) (stroke (width 0.15) (type default)))
+(gr_line (start 184.2174451 88.9063712166168) (end 202.52456117575397 99.47598961084917) (layer Edge.Cuts) (stroke (width 0.15) (type default)))
+(gr_line (start 202.2394151295069 100.4077655075903) (end 185.55536086521693 99.23210059556159) (layer Edge.Cuts) (stroke (width 0.15) (type default)))
+(gr_line (start 185.1362133148852 100.0510869874045) (end 211.0531597636026 131.12986674538013) (layer Edge.Cuts) (stroke (width 0.15) (type default)))
+(gr_line (start 211.02271165951797 131.803643340482) (end 198.27245950682325 144.55389549317673) (layer Edge.Cuts) (stroke (width 0.15) (type default)))
 (gr_line (start 197.5573001306715 144.5456552181502) (end 185.2184018103768 131.6245719172887) (layer Edge.Cuts) (stroke (width 0.15) (type default)))
 (gr_line (start 185.11474537091743 131.54156036435938) (end 167.73632242747522 121.07577102297391) (layer Edge.Cuts) (stroke (width 0.15) (type default)))
-(gr_line (start 167.61101352447525 121.02201021014679) (end 149.67542832928424 116.0872276331902) (layer Edge.Cuts) (stroke (width 0.15) (type default)))
-(gr_line (start 149.32552987561743 115.73612318902917) (end 145.83984366392013 102.89472334271511) (layer Edge.Cuts) (stroke (width 0.15) (type default)))
-(gr_line (start 145.28816068340882 102.53050838832783) (end 92.4425969819845 109.90929922465821) (layer Edge.Cuts) (stroke (width 0.15) (type default)))
+(gr_line (start 167.61101352447525 121.02201021014679) (end 149.710817093128 116.09696446939239) (layer Edge.Cuts) (stroke (width 0.15) (type default)))
+(gr_line (start 149.3496706345805 115.69345582742767) (end 146.44949553337028 97.46837645346864) (layer Edge.Cuts) (stroke (width 0.15) (type default)))
+(gr_line (start 145.97070169267394 97.04717810078023) (end 108.98268763536329 95.93753767906091) (layer Edge.Cuts) (stroke (width 0.15) (type default)))
+(gr_line (start 108.4732258911544 96.51148092941446) (end 110.21182009800681 108.10245993570732) (layer Edge.Cuts) (stroke (width 0.15) (type default)))
+(gr_line (start 109.75389440169705 108.67529078487426) (end 92.41291032810221 109.9460646235092) (layer Edge.Cuts) (stroke (width 0.15) (type default)))
 (gr_arc (start 87.51811424775414 53.90547845501909) (mid 87.17664344775413 54.0812949550191) (end 87.06061104775414 54.4474235550191) (layer Edge.Cuts) (stroke (width 0.15) (type default)))
 (gr_arc (start 108.5050376 52.19601094933076) (mid 108.83207 52.03655944933076) (end 108.964445 51.69766144933076) (layer Edge.Cuts) (stroke (width 0.15) (type default)))
@@
 (gr_arc (start 183.96667038015485 43.26992130875763) (mid 183.81748338015484 42.91387050875763) (end 183.45917118015484 42.770199508757635) (layer Edge.Cuts) (stroke (width 0.15) (type default)))
 (gr_arc (start 183.9674451 45.01481240004068) (mid 183.9674451 45.014701400040686) (end 183.9674451 45.01459040004068) (layer Edge.Cuts) (stroke (width 0.15) (type default)))
-(gr_arc (start 183.9674451 93.93435851661681) (mid 184.0344324 94.18435851661681) (end 184.2174451 94.36737121661682) (layer Edge.Cuts) (stroke (width 0.15) (type default)))
-(gr_arc (start 204.45659455980976 106.21974155985939) (mid 204.37021085980976 106.0460345598594) (end 204.22421145980977 105.91828315985939) (layer Edge.Cuts) (stroke (width 0.15) (type default)))
-(gr_arc (start 211.14051951990055 131.68583548009963) (mid 211.27021541990055 131.46061828009962) (end 211.26934921990053 131.20072768009962) (layer Edge.Cuts) (stroke (width 0.15) (type default)))
+(gr_arc (start 183.9674451 88.4733585166168) (mid 184.0344324 88.7233585166168) (end 184.2174451 88.9063712166168) (layer Edge.Cuts) (stroke (width 0.15) (type default)))
+(gr_arc (start 202.23941517575395 100.40776551084916) (mid 202.75267427575395 100.05531651084917) (end 202.52456107575395 99.47598961084915) (layer Edge.Cuts) (stroke (width 0.15) (type default)))
+(gr_arc (start 185.5553608189699 99.23210059230273) (mid 185.0751196189699 99.50306939230273) (end 185.1362134189699 100.05108699230273) (layer Edge.Cuts) (stroke (width 0.15) (type default)))
+(gr_arc (start 211.02271165951794 131.80364334048198) (mid 211.16864855951792 131.47266194048197) (end 211.05315975951794 131.129866740482) (layer Edge.Cuts) (stroke (width 0.15) (type default)))
 (gr_arc (start 197.55730020682324 144.5456551931767) (mid 197.91314540682325 144.70030889317673) (end 198.27245950682325 144.5538953931767) (layer Edge.Cuts) (stroke (width 0.15) (type default)))
 (gr_arc (start 185.21840173422504 131.62457194226215) (mid 185.16934173422504 131.57960944226215) (end 185.11474533422503 131.54156034226216) (layer Edge.Cuts) (stroke (width 0.15) (type default)))
 (gr_arc (start 167.7363223907828 121.07577100087666) (mid 167.6755091907828 121.04459890087666) (end 167.6110134907828 121.02201020087666) (layer Edge.Cuts) (stroke (width 0.15) (type default)))
-(gr_arc (start 149.32552986297674 115.73612314246033) (mid 149.45390776297674 115.95808674246032) (end 149.67542826297674 116.08722764246032) (layer Edge.Cuts) (stroke (width 0.15) (type default)))
-(gr_arc (start 145.83984367656083 102.89472338928387) (mid 145.63278067656083 102.60843598928388) (end 145.28816067656084 102.53050828928387) (layer Edge.Cuts) (stroke (width 0.15) (type default)))
-(gr_arc (start 91.87535728883246 109.45769882370203) (mid 92.06202788883246 109.80527372370203) (end 92.44259698883246 109.90929922370204) (layer Edge.Cuts) (stroke (width 0.15) (type default)))
+(gr_arc (start 149.34967062682045 115.69345577866251) (mid 149.47088862682045 115.94833397866252) (end 149.71081702682045 116.09696447866251) (layer Edge.Cuts) (stroke (width 0.15) (type default)))
+(gr_arc (start 146.44949554113035 97.46837650223388) (mid 146.28596044113036 97.17154200223388) (end 145.97070174113034 97.04717810223387) (layer Edge.Cuts) (stroke (width 0.15) (type default)))
+(gr_arc (start 108.98268768381968 95.9375376805146) (mid 108.59376008381967 96.1053893805146) (end 108.47322578381967 96.5114808805146) (layer Edge.Cuts) (stroke (width 0.15) (type default)))
+(gr_arc (start 109.75389440534157 108.6752907846072) (mid 110.10789870534157 108.4888344846072) (end 110.21182010534156 108.1024599846072) (layer Edge.Cuts) (stroke (width 0.15) (type default)))
+(gr_arc (start 91.87827173174674 109.49099742324213) (mid 92.05228523174674 109.82815192324213) (end 92.41291033174674 109.94606462324214) (layer Edge.Cuts) (stroke (width 0.15) (type default)))
 (gr_line (start 93.6367273 107.5834531) (end 107.5834531 106.3632727) (layer Edge.Cuts) (stroke (width 0.15) (type default)))
 (gr_line (start 107.5834531 106.3632727) (end 106.3632727 92.4165469) (layer Edge.Cuts) (stroke (width 0.15) (type default)))
